File: schematics/generic_fogger_timer/generic_fogger_timer.kicad_sch (KiCad schematic)
At the start: 36 parts, among them J1 IEC-60320 E Conn, SW4 "Power", SW5 "Manual", SW6 "Timer", U1 MOC3023M, U2 CD4541B, U3 CD4541B

Commit message: Triple checking how the basic wired remotes work with fog machines.
Other:
- title: Generic Fog Machine Timer -> Common Fog Machine Timer
Changed lines of the file:
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@@
   (paper "USLetter")
   (title_block
-    (title "Generic Fog Machine Timer")
+    (title "Common Fog Machine Timer")
     (comment 1 "FWC-4B.PCB Rev 3")
-    (comment 2 "Schematic for educational purposes only")
+    (comment 2 "To understand how to interface to common \"party-store\" consumer fog machines.")
   )
   (junction (at 142.494 67.564) (diameter 0) (color 0 0 0 0)
